Commit message: Add files via upload

File: misty_description/urdf/misty.xacro (robot description, xacro)
@@ -3,4 +3,6 @@
 <xacro:include filename="$(find misty_description)/urdf/misty.trans" />
 <xacro:include filename="$(find misty_description)/urdf/misty.gazebo" />
+<xacro:include filename="$(find misty_description)/urdf/misty_gazebo_plugins.xacro"/>
+<xacro:property name="camera_link" value="0.05" />
 <material name="silver">
   <color rgba="0.700 0.700 0.700 1.000"/>
@@ -28,10 +30,10 @@
 <link name="MIDDLE_LEFT_WHEEL_1">
   <inertial>
-    <origin rpy="0 0 0" xyz="0.37532252073471667 0.07491599608036578 -0.11963838591658377"/>
+    <origin rpy="0 0 0" xyz="0 0 0"/>
     <mass value="0.008942480656590288"/>
     <inertia ixx="1e-06" ixy="0.0" ixz="0.0" iyy="2e-06" iyz="0.0" izz="1e-06"/>
   </inertial>
   <visual>
-    <origin rpy="0 0 0" xyz="0.382014 0.006691 -0.147284"/>
+    <origin rpy="0 0 0" xyz="0.006691 -0.060225 -0.027646"/>
     <geometry>
       <mesh filename="package://misty_description/meshes/MIDDLE_LEFT_WHEEL_1.stl" scale="0.001 0.001 0.001"/>
@@ -40,7 +42,7 @@
   </visual>
   <collision>
-    <origin rpy="0 0 0" xyz="0.382014 0.006691 -0.147284"/>
-    <geometry>
-      <mesh filename="package://misty_description/meshes/MIDDLE_LEFT_WHEEL_1.stl" scale="0.001 0.001 0.001"/>
+    <origin rpy="0 0 0" xyz="0.008579863636 -0.0739125 -0.0339291812"/>
+    <geometry>
+      <mesh filename="package://misty_description/meshes/MIDDLE_LEFT_WHEEL_1.stl" scale="0.0012272727 0.0012272727 0.0012272727"/>
     </geometry>
   </collision>
@@ -48,10 +50,10 @@
 <link name="REAR_LEFT_WHEEL_1">
   <inertial>
-    <origin rpy="0 0 0" xyz="0.30682252073471655 0.14341599608042296 -0.11963838591658374"/>
+    <origin rpy="0 0 0" xyz="0 0 0"/>
     <mass value="0.008942480656590273"/>
     <inertia ixx="1e-06" ixy="0.0" ixz="-0.0" iyy="2e-06" iyz="0.0" izz="1e-06"/>
   </inertial>
   <visual>
-    <origin rpy="0 0 0" xyz="0.382014 0.075191 -0.147284"/>
+    <origin rpy="0 0 0" xyz="0.075191 -0.060225 -0.027646"/>
     <geometry>
       <mesh filename="package://misty_description/meshes/REAR_LEFT_WHEEL_1.stl" scale="0.001 0.001 0.001"/>
@@ -60,7 +62,7 @@
   </visual>
   <collision>
-    <origin rpy="0 0 0" xyz="0.382014 0.075191 -0.147284"/>
-    <geometry>
-      <mesh filename="package://misty_description/meshes/REAR_LEFT_WHEEL_1.stl" scale="0.001 0.001 0.001"/>
+    <origin rpy="0 0 0" xyz="0.09227986364 -0.0739125 -0.03392918182"/>
+    <geometry>
+      <mesh filename="package://misty_description/meshes/REAR_LEFT_WHEEL_1.stl" scale="0.0012272727 0.0012272727 0.0012272727"/>
     </geometry>
   </collision>
@@ -68,10 +70,10 @@
 <link name="REAR_RIGHT_WHEEL_1">
   <inertial>
-    <origin rpy="0 0 0" xyz="0.18562252073468966 0.0069659960804353965 -0.11963838591658374"/>
+    <origin rpy="0 0 0" xyz="0 0 0"/>
     <mass value="0.008942480656590273"/>
     <inertia ixx="1e-06" ixy="-0.0" ixz="0.0" iyy="2e-06" iyz="-0.0" izz="1e-06"/>
   </inertial>
   <visual>
-    <origin rpy="0 0 0" xyz="0.260814 0.075191 -0.147284"/>
+    <origin rpy="0 0 0" xyz="0.075191 0.060225 -0.027646"/>
     <geometry>
       <mesh filename="package://misty_description/meshes/REAR_RIGHT_WHEEL_1.stl" scale="0.001 0.001 0.001"/>
@@ -80,7 +82,7 @@
   </visual>
   <collision>
-    <origin rpy="0 0 0" xyz="0.260814 0.075191 -0.147284"/>
-    <geometry>
-      <mesh filename="package://misty_description/meshes/REAR_RIGHT_WHEEL_1.stl" scale="0.001 0.001 0.001"/>
+    <origin rpy="0 0 0" xyz="0.09227986364 0.0739125 -0.03392918182"/>
+    <geometry>
+      <mesh filename="package://misty_description/meshes/REAR_RIGHT_WHEEL_1.stl" scale="0.0012272727 0.0012272727 0.0012272727"/>
     </geometry>
   </collision>
@@ -88,10 +90,10 @@
 <link name="MIDDLE_RIGHT_WHEEL_1">
   <inertial>
-    <origin rpy="0 0 0" xyz="0.2541225207346897 -0.06153400391956494 -0.11963838591658375"/>
+    <origin rpy="0 0 0" xyz="0 0 0"/>
     <mass value="0.008942480656590271"/>
     <inertia ixx="1e-06" ixy="-0.0" ixz="0.0" iyy="2e-06" iyz="0.0" izz="1e-06"/>
   </inertial>
   <visual>
-    <origin rpy="0 0 0" xyz="0.260814 0.006691 -0.147284"/>
+    <origin rpy="0 0 0" xyz="0.006691 0.060225 -0.027646"/>
     <geometry>
       <mesh filename="package://misty_description/meshes/MIDDLE_RIGHT_WHEEL_1.stl" scale="0.001 0.001 0.001"/>
@@ -100,7 +102,7 @@
   </visual>
   <collision>
-    <origin rpy="0 0 0" xyz="0.260814 0.006691 -0.147284"/>
-    <geometry>
-      <mesh filename="package://misty_description/meshes/MIDDLE_RIGHT_WHEEL_1.stl" scale="0.001 0.001 0.001"/>
+    <origin rpy="0 0 0" xyz="0.008579863636 0.0739125 -0.0339291812"/>
+    <geometry>
+      <mesh filename="package://misty_description/meshes/MIDDLE_RIGHT_WHEEL_1.stl" scale="0.0012272727 0.0012272727 0.0012272727"/>
     </geometry>
   </collision>
@@ -348,5 +350,5 @@
 <link name="LEFT_ARM_1">
   <inertial>
-    <origin rpy="0 0 0" xyz="0.02912463794527921 0.013529199094012623 -0.008524139150373061"/>
+    <origin rpy="0 0 0" xyz="0.015 0 0"/>
     <mass value="0.031754892803095174"/>
     <inertia ixx="1.4e-05" ixy="-5e-06" ixz="8e-06" iyy="2.8e-05" iyz="3e-06" izz="2e-05"/>
@@ -368,5 +370,5 @@
 <link name="RIGHT_ARM_1">
   <inertial>
-    <origin rpy="0 0 0" xyz="0.028999453853953583 -0.01685124115287527 -0.011525075237750232"/>
+    <origin rpy="0 0 0" xyz="0.015 0 0"/>
     <mass value="0.03134177021944716"/>
     <inertia ixx="1.5e-05" ixy="4e-06" ixz="8e-06" iyy="2.7e-05" iyz="-3e-06" izz="1.8e-05"/>
@@ -408,5 +410,5 @@
 <link name="RIGHT_ARM_CONNECTOR_1">
   <inertial>
-    <origin rpy="0 0 0" xyz="0.00018193452656749265 -0.00652324319868379 -8.322442592700874e-05"/>
+    <origin rpy="0 0 0" xyz="0 0 0"/>
     <mass value="0.027172748965990867"/>
     <inertia ixx="2e-06" ixy="0.0" ixz="0.0" iyy="3e-06" iyz="-0.0" izz="2e-06"/>
@@ -428,5 +430,5 @@
 <link name="LEFT_ARM_CONNECTOR_1">
   <inertial>
-    <origin rpy="0 0 0" xyz="0.0001670098430530155 0.006523521945876604 -8.215617760007343e-05"/>
+    <origin rpy="0 0 0" xyz="0 0 0"/>
     <mass value="0.027172549960048142"/>
     <inertia ixx="2e-06" ixy="-0.0" ixz="0.0" iyy="3e-06" iyz="0.0" izz="2e-06"/>
@@ -448,10 +450,10 @@
 <link name="FRONT_LEFT_WHEEL_1">
   <inertial>
-    <origin rpy="0 0 0" xyz="0.4352225186156042 0.011728209281953311 -0.1196382849296091"/>
+    <origin rpy="0 0 0" xyz="0 0 0"/>
     <mass value="0.025418776956642474"/>
     <inertia ixx="5e-06" ixy="0.0" ixz="0.0" iyy="8e-06" iyz="-0.0" izz="5e-06"/>
   </inertial>
   <visual>
-    <origin rpy="0 0 0" xyz="0.374914 -0.060309 -0.154784"/>
+    <origin rpy="0 0 0" xyz="-0.060309 -0.060225 -0.035146"/>
     <geometry>
       <mesh filename="package://misty_description/meshes/FRONT_LEFT_WHEEL_1.stl" scale="0.001 0.001 0.001"/>
@@ -460,7 +462,7 @@
   </visual>
   <collision>
-    <origin rpy="0 0 0" xyz="0.374914 -0.060309 -0.154784"/>
-    <geometry>
-      <mesh filename="package://misty_description/meshes/FRONT_LEFT_WHEEL_1.stl" scale="0.001 0.001 0.001"/>
+    <origin rpy="0 0 0" xyz="-0.07053086441 -0.07043262712 -0.04110294915"/>
+    <geometry>
+      <mesh filename="package://misty_description/meshes/FRONT_LEFT_WHEEL_1.stl" scale="0.001169491525 0.001169491525 0.001169491525"/>
     </geometry>
   </collision>
@@ -468,10 +470,10 @@
 <link name="FRONT_RIGHT_WHEEL_1">
   <inertial>
-    <origin rpy="0 0 0" xyz="0.32822251861559876 -0.13234621712115296 -0.11963828492960912"/>
+    <origin rpy="0 0 0" xyz="0 0 0"/>
     <mass value="0.0254187769566425"/>
     <inertia ixx="5e-06" ixy="-0.0" ixz="-0.0" iyy="8e-06" iyz="0.0" izz="5e-06"/>
   </inertial>
   <visual>
-    <origin rpy="0 0 0" xyz="0.267914 -0.060309 -0.154784"/>
+    <origin rpy="0 0 0" xyz="-0.060309 0.060225 -0.035146"/>
     <geometry>
       <mesh filename="package://misty_description/meshes/FRONT_RIGHT_WHEEL_1.stl" scale="0.001 0.001 0.001"/>
@@ -480,12 +482,38 @@
   </visual>
   <collision>
-    <origin rpy="0 0 0" xyz="0.267914 -0.060309 -0.154784"/>
-    <geometry>
-      <mesh filename="package://misty_description/meshes/FRONT_RIGHT_WHEEL_1.stl" scale="0.001 0.001 0.001"/>
-    </geometry>
-  </collision>
-</link>
+    <origin rpy="0 0 0" xyz="-0.07053086441 0.07043262712 -0.04110294915"/>
+    <geometry>
+      <mesh filename="package://misty_description/meshes/FRONT_RIGHT_WHEEL_1.stl" scale="0.001169491525 0.001169491525 0.001169491525"/>
+    </geometry>
+  </collision>
+</link>
+<link name="camera_link">
+  <collision>
+    <origin xyz = "0.07 0 0.05" rpy="0 0 0"/>
+    <geometry>
+  <box size="${camera_link} ${camera_link} ${camera_link}"/>
+   </geometry>
+  </collision>
+  <visual>
+    <origin xyz="0.07 0 0.05" rpy="0 0 0"/>
+    <geometry>
+  <box size="${camera_link} ${camera_link} ${camera_link}"/>
+    </geometry>
+    <material name="blue"/>
+  </visual>
+  <inertial>
+    <mass value="1e-5" />
+    <origin xyz="0.07 0 0.05" rpy="0 0 0"/>
+    <intertia ixx="1e-6" ixy="0" ixz="0" iyy="1e-6" iyz="0" izz="1e-6" />
+  </inertial>
+</link>
+<joint name = "camera_joint" type="fixed">
+  <axis xyz="0.07 0 0.05" />
+  <origin xyz="${camera_link} 0 0" rpy="0 0 0"/>
+  <parent link="HEAD_1"/>
+  <child link="camera_link"/>
+</joint>
 <joint name="Rev2" type="continuous">
-  <origin rpy="0 0 0" xyz="-0.382014 -0.006691 0.147284"/>
+  <origin rpy="0 0 0" xyz="-0.006691 0.060225 0.028646"/>
   <parent link="base_link"/>
   <child link="MIDDLE_LEFT_WHEEL_1"/>
@@ -493,5 +521,5 @@
 </joint>
 <joint name="Rev3" type="continuous">
-  <origin rpy="0 0 0" xyz="-0.382014 -0.075191 0.147284"/>
+  <origin rpy="0 0 0" xyz="-0.075191 0.060225 0.028646"/>
   <parent link="base_link"/>
   <child link="REAR_LEFT_WHEEL_1"/>
@@ -499,5 +527,5 @@
 </joint>
 <joint name="Rev4" type="continuous">
-  <origin rpy="0 0 0" xyz="-0.260814 -0.075191 0.147284"/>
+  <origin rpy="0 0 0" xyz="-0.075191 -0.060225 0.028646"/>
   <parent link="base_link"/>
   <child link="REAR_RIGHT_WHEEL_1"/>
@@ -505,5 +533,5 @@
 </joint>
 <joint name="Rev5" type="continuous">
-  <origin rpy="0 0 0" xyz="-0.260814 -0.006691 0.147284"/>
+  <origin rpy="0 0 0" xyz="-0.006691 -0.060225 0.028646"/>
   <parent link="base_link"/>
   <child link="MIDDLE_RIGHT_WHEEL_1"/>
@@ -598,5 +626,5 @@
 </joint>
 <joint name="Rev37" type="continuous">
-  <origin rpy="0 0 0" xyz="-0.374914 0.060309 0.154784"/>
+  <origin rpy="0 0 0" xyz="0.060309 0.060225 0.036146"/>
   <parent link="base_link"/>
   <child link="FRONT_LEFT_WHEEL_1"/>
@@ -604,8 +632,8 @@
 </joint>
 <joint name="Rev38" type="continuous">
-  <origin rpy="0 0 0" xyz="-0.267914 0.060309 0.154784"/>
+  <origin rpy="0 0 0" xyz="0.060309 -0.060225 0.036146"/>
   <parent link="base_link"/>
   <child link="FRONT_RIGHT_WHEEL_1"/>
-  <axis xyz="-0.0 -1.0 -0.0"/>
+  <axis xyz="-0.0 1.0 -0.0"/>
 </joint>
 </robot>

Commit message: Add files via upload

File: misty_description/urdf/misty.xacro (robot description, xacro)
@@ -350,5 +350,5 @@
 <link name="LEFT_ARM_1">
   <inertial>
-    <origin rpy="0 0 0" xyz="0.015 0 0"/>
+    <origin rpy="0 0 0" xyz="0.013297 0 0.001514"/>
     <mass value="0.031754892803095174"/>
     <inertia ixx="1.4e-05" ixy="-5e-06" ixz="8e-06" iyy="2.8e-05" iyz="3e-06" izz="2e-05"/>
@@ -370,5 +370,5 @@
 <link name="RIGHT_ARM_1">
   <inertial>
-    <origin rpy="0 0 0" xyz="0.015 0 0"/>
+    <origin rpy="0 0 0" xyz="0.014964 0 0.000287"/>
     <mass value="0.03134177021944716"/>
     <inertia ixx="1.5e-05" ixy="4e-06" ixz="8e-06" iyy="2.7e-05" iyz="-3e-06" izz="1.8e-05"/>

Commit message: Add files via upload

File: misty_description/urdf/misty.xacro (robot description, xacro)
@@ -31,5 +31,5 @@
   <inertial>
     <origin rpy="0 0 0" xyz="0 0 0"/>
-    <mass value="0.008942480656590288"/>
+    <mass value="0.00008942480656590271"/>
     <inertia ixx="1e-06" ixy="0.0" ixz="0.0" iyy="2e-06" iyz="0.0" izz="1e-06"/>
   </inertial>
@@ -41,15 +41,15 @@
     <material name="silver"/>
   </visual>
-  <collision>
+  <!--collision>
     <origin rpy="0 0 0" xyz="0.008579863636 -0.0739125 -0.0339291812"/>
     <geometry>
       <mesh filename="package://misty_description/meshes/MIDDLE_LEFT_WHEEL_1.stl" scale="0.0012272727 0.0012272727 0.0012272727"/>
     </geometry>
-  </collision>
+  </collision!-->
 </link>
 <link name="REAR_LEFT_WHEEL_1">
   <inertial>
     <origin rpy="0 0 0" xyz="0 0 0"/>
-    <mass value="0.008942480656590273"/>
+    <mass value="0.00008942480656590273"/>
     <inertia ixx="1e-06" ixy="0.0" ixz="-0.0" iyy="2e-06" iyz="0.0" izz="1e-06"/>
   </inertial>
@@ -61,15 +61,15 @@
     <material name="silver"/>
   </visual>
-  <collision>
+  <!--collision>
     <origin rpy="0 0 0" xyz="0.09227986364 -0.0739125 -0.03392918182"/>
     <geometry>
       <mesh filename="package://misty_description/meshes/REAR_LEFT_WHEEL_1.stl" scale="0.0012272727 0.0012272727 0.0012272727"/>
     </geometry>
-  </collision>
+  </collision-->
 </link>
 <link name="REAR_RIGHT_WHEEL_1">
   <inertial>
     <origin rpy="0 0 0" xyz="0 0 0"/>
-    <mass value="0.008942480656590273"/>
+    <mass value="0.00008942480656590273"/>
     <inertia ixx="1e-06" ixy="-0.0" ixz="0.0" iyy="2e-06" iyz="-0.0" izz="1e-06"/>
   </inertial>
@@ -81,8 +81,29 @@
     <material name="silver"/>
   </visual>
-  <collision>
-    <origin rpy="0 0 0" xyz="0.09227986364 0.0739125 -0.03392918182"/>
-    <geometry>
-      <mesh filename="package://misty_description/meshes/REAR_RIGHT_WHEEL_1.stl" scale="0.0012272727 0.0012272727 0.0012272727"/>
+  <!--collision>
+    <origin rpy="0 0 0" xyz="0.0 0.0 0.0"/>
+    <geometry>
+      <mesh filename="package://misty_description/meshes/REAR_RIGHT_WHEEL_1.stl" scale="0.0012272727 0.0012272727 0.0012272727">
+    </geometry>
+  </collision-->
+</link>
+<link name="BALANCE_WHEEL">
+  <inertial>
+    <origin rpy="0 0 0" xyz="0 0 0"/>
+    <mass value="0.01788496131"/>
+    <inertia ixx="1e-06" ixy="-0.0" ixz="0.0" iyy="2e-06" iyz="-0.0" izz="1e-06"/>
+  </inertial>
+  <!--visual>
+    <origin rpy="0 0 0" xyz="0.075191 0.0 -0.027646"/>
+    <geometry>
+      <mesh filename="package://misty_description/meshes/REAR_RIGHT_WHEEL_1.stl" scale="0.001 0.001 0.001"/>
+    </geometry>
+    <material name="silver"/>
+  </visual-->
+  <collision>
+    <origin rpy="0 0 0" xyz="0.0 0.0 0.0"/>
+    <geometry>
+      <sphere radius = "0.027"/>
+      <!--mesh filename="package://misty_description/meshes/REAR_RIGHT_WHEEL_1.stl" scale="0.0012272727 0.0012272727 0.0012272727"/-->
     </geometry>
   </collision>
@@ -91,5 +112,5 @@
   <inertial>
     <origin rpy="0 0 0" xyz="0 0 0"/>
-    <mass value="0.008942480656590271"/>
+    <mass value="0.00008942480656590271"/>
     <inertia ixx="1e-06" ixy="-0.0" ixz="0.0" iyy="2e-06" iyz="0.0" izz="1e-06"/>
   </inertial>
@@ -101,10 +122,10 @@
     <material name="silver"/>
   </visual>
-  <collision>
+  <!--collision>
     <origin rpy="0 0 0" xyz="0.008579863636 0.0739125 -0.0339291812"/>
     <geometry>
       <mesh filename="package://misty_description/meshes/MIDDLE_RIGHT_WHEEL_1.stl" scale="0.0012272727 0.0012272727 0.0012272727"/>
     </geometry>
-  </collision>
+  </collision-->
 </link>
 <link name="BODY_BASE_CONNECTOR_1">
@@ -151,5 +172,5 @@
   <inertial>
     <origin rpy="0 0 0" xyz="-0.07255561628768126 0.027216822680745684 -0.00903210537434923"/>
-    <mass value="0.14825796927747048"/>
+    <mass value="0.14768918703590395"/>
     <inertia ixx="0.000172" ixy="-2.5e-05" ixz="7.5e-05" iyy="0.000855" iyz="4.1e-05" izz="0.000793"/>
   </inertial>
@@ -371,5 +392,5 @@
   <inertial>
     <origin rpy="0 0 0" xyz="0.014964 0 0.000287"/>
-    <mass value="0.03134177021944716"/>
+    <mass value="0.031754892803095174"/>
     <inertia ixx="1.5e-05" ixy="4e-06" ixz="8e-06" iyy="2.7e-05" iyz="-3e-06" izz="1.8e-05"/>
   </inertial>
@@ -431,5 +452,5 @@
   <inertial>
     <origin rpy="0 0 0" xyz="0 0 0"/>
-    <mass value="0.027172549960048142"/>
+    <mass value="0.027172748965990867"/>
     <inertia ixx="2e-06" ixy="-0.0" ixz="0.0" iyy="3e-06" iyz="0.0" izz="2e-06"/>
   </inertial>
@@ -462,7 +483,8 @@
   </visual>
   <collision>
-    <origin rpy="0 0 0" xyz="-0.07053086441 -0.07043262712 -0.04110294915"/>
-    <geometry>
-      <mesh filename="package://misty_description/meshes/FRONT_LEFT_WHEEL_1.stl" scale="0.001169491525 0.001169491525 0.001169491525"/>
+    <origin rpy="1.570796327 0 0" xyz="0 0.008 0"/>
+    <geometry>
+      <cylinder length="0.024" radius="0.0345"/>
+      <!--mesh filename="package://misty_description/meshes/FRONT_LEFT_WHEEL_1.stl" scale="0.001169491525 0.001169491525 0.001169491525"/-->
     </geometry>
   </collision>
@@ -471,5 +493,5 @@
   <inertial>
     <origin rpy="0 0 0" xyz="0 0 0"/>
-    <mass value="0.0254187769566425"/>
+    <mass value="0.025418776956642474"/>
     <inertia ixx="5e-06" ixy="-0.0" ixz="-0.0" iyy="8e-06" iyz="0.0" izz="5e-06"/>
   </inertial>
@@ -482,7 +504,8 @@
   </visual>
   <collision>
-    <origin rpy="0 0 0" xyz="-0.07053086441 0.07043262712 -0.04110294915"/>
-    <geometry>
-      <mesh filename="package://misty_description/meshes/FRONT_RIGHT_WHEEL_1.stl" scale="0.001169491525 0.001169491525 0.001169491525"/>
+    <origin rpy="1.570796327 0 0" xyz="0 -0.008 0"/>
+    <geometry>
+      <!--mesh filename="package://misty_description/meshes/FRONT_RIGHT_WHEEL_1.stl" scale="0.001169491525 0.001169491525 0.001169491525"/-->
+      <cylinder length="0.024" radius="0.0345"/>
     </geometry>
   </collision>
@@ -637,3 +660,9 @@
   <axis xyz="-0.0 1.0 -0.0"/>
 </joint>
+<joint name="Rev39" type="continuous">
+  <origin rpy="0 0 0" xyz="-0.075191 -0.0 0.028646"/>
+  <parent link="base_link"/>
+  <child link="BALANCE_WHEEL"/>
+  <axis xyz="0 1.0 0"/>
+</joint>
 </robot>

Commit message: Add files via upload

File: misty_description/urdf/misty.xacro (robot description, xacro)
@@ -531,4 +531,24 @@
   </inertial>
 </link>
+<link name="imu_sensor_link">
+  <collision>
+    <origin xyz="0 0 0" rpy="0 0 0"/>
+    <geometry>
+      <box size="0.02 0.02 0.02"/>
+    </geometry>
+  </collision>
+  <visual>
+    <origin xyz="0 0 0" rpy="0 0 0"/>
+    <geometry>
+      <box size="0.02 0.02 0.02"/>
+    </geometry>
+    <material name="iRobot/Red"/>
+  </visual>
+  <inertial>
+    <mass value="0.001" />
+    <origin xyz="0 0 0" rpy="0 0 0"/>
+      <inertia ixx="0.00000015" ixy="0" ixz="0" iyy="0.00000015" iyz="0" izz="0.00000015" />
+  </inertial>
+</link>
 <joint name = "camera_joint" type="fixed">
   <axis xyz="0.07 0 0.05" />
@@ -537,4 +557,10 @@
   <child link="camera_link"/>
 </joint>
+<joint name="imu_sensor_joint" type="fixed">
+  <axis xyz="0 0 1" />
+  <origin xyz="0 0 0" rpy="0 0 0"/>
+  <parent link="base_link"/>
+  <child link="imu_sensor_link"/>
+</joint>
 <joint name="Rev2" type="continuous">
   <origin rpy="0 0 0" xyz="-0.006691 0.060225 0.028646"/>

File: misty_description/urdf/misty_gazebo_plugins.xacro (robot description, xacro)
@@ -40,23 +40,21 @@
       </sensor>
    </gazebo>
-  <gazebo reference="imu_link">
-    <gravity>true</gravity>
-    <sensor name="imu_sensor" type="imu">
-      <always_on>true</always_on>
-      <update_rate>100</update_rate>
-      <visualize>true</visualize>
-      <topic>__default_topic__</topic>
-      <plugin filename="libgazebo_ros_imu_sensor.so" name="imu_plugin">
-        <topicName>imu</topicName>
-        <bodyName>imu_link</bodyName>
-        <updateRateHZ>10.0</updateRateHZ>
-        <gaussianNoise>0.0</gaussianNoise>
-        <xyzOffset>0 0 0</xyzOffset>
-        <rpyOffset>0 0 0</rpyOffset>
-        <frameName>imu_link</frameName>
-        <initialOrientationAsReference>false</initialOrientationAsReference>
-      </plugin>
-      <pose>0 0 0 0 0 0</pose>
-    </sensor>
-  </gazebo>
+  <gazebo reference="imu_sensor_link">
+  <gravity>true</gravity>
+  <sensor name='imu_sensor' type='imu'>
+    <always_on>1</always_on>
+    <update_rate>1000</update_rate>
+    <visualize>1</visualize>
+    <topic>misty_imu</topic>
+    <plugin name='imu_plugin' filename='libgazebo_ros_imu_sensor.so'>
+      <topicName>imu_data</topicName>
+      <frameName>imu_sensor_link</frameName>
+      <updateRateHZ>10.0</updateRateHZ>
+      <gaussianNoise>0.0</gaussianNoise>
+      <xyzOffset>0 0 0</xyzOffset>
+      <rpyOffset>0 0 0</rpyOffset>
+    </plugin>
+    <pose>0 0 0 0 0 0</pose>
+  </sensor>
+</gazebo>
 </robot>
